File: rtd_board/_autosave-rtd_board.kicad_sch (KiCad schematic)
At the start: 15 parts

Commit message: more RTD changes
Connections:
- net +3V3: now also U?.12 (VCC), U?.17 (VDD), U?.9 (VDD)
- net GND: now also U?.10 (GND), U?.11 (GND), U?.16 (GND)
- net IO_EXP_SDA: now reaches U?.13 (SDA)
- net IO_EXP_SCL: now reaches U?.14 (SCL)
Other:
- note added: "Address: 0x70"
Changed lines of the file:
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@@
   (no_connect (at 26.67 25.4))
   (no_connect (at 91.44 76.2))
+  (wire (pts (xy 254 59.69) (xy 254 72.39))
+    (stroke (width 0) (type default) (color 0 0 0 0))
+  )
   (wire (pts (xy 180.34 85.09) (xy 190.5 85.09))
     (stroke (width 0) (type default) (color 0 0 0 0))
@@
     (stroke (width 0) (type default) (color 0 0 0 0))
   )
+  (wire (pts (xy 275.59 72.39) (xy 275.59 62.23))
+    (stroke (width 0) (type default) (color 0 0 0 0))
+  )
   (wire (pts (xy 190.5 90.17) (xy 177.8 90.17))
     (stroke (width 0) (type default) (color 0 0 0 0))
@@
     (stroke (width 0) (type default) (color 0 0 0 0))
   )
+  (wire (pts (xy 270.51 48.26) (xy 274.32 48.26))
+    (stroke (width 0) (type default) (color 0 0 0 0))
+  )
+  (wire (pts (xy 238.76 48.26) (xy 242.57 48.26))
+    (stroke (width 0) (type default) (color 0 0 0 0))
+  )
   (wire (pts (xy 177.8 90.17) (xy 177.8 97.79))
     (stroke (width 0) (type default) (color 0 0 0 0))
   )
+  (wire (pts (xy 254 72.39) (xy 275.59 72.39))
+    (stroke (width 0) (type default) (color 0 0 0 0))
+  )
   (wire (pts (xy 180.34 85.09) (xy 180.34 92.71))
     (stroke (width 0) (type default) (color 0 0 0 0))
@@
     (effects (font (size 1.27 1.27)) (justify left bottom))
   )
+  (text "Address: 0x70" (at 250.19 19.05 0)
+    (effects (font (size 1.27 1.27)) (justify left bottom))
+  )
   (text "RTD 6\n" (at 119.38 86.36 0)
     (effects (font (size 1.27 1.27)) (justify left bottom))
@@
     (effects (font (size 1.27 1.27)) (justify left bottom))
   )
+  (label "IO_EXP_SCL" (at 259.08 59.69 270)
+    (effects (font (size 1.27 1.27)) (justify right bottom))
+  )
   (label "RTD3_F+" (at 111.76 33.02 180)
     (effects (font (size 1.27 1.27)) (justify right bottom))
@@
   (label "RTD2_SCK" (at 90.17 29.21 0)
     (effects (font (size 1.27 1.27)) (justify left bottom))
+  )
+  (label "IO_EXP_SDA" (at 256.54 59.69 270)
+    (effects (font (size 1.27 1.27)) (justify right bottom))
   )
   (label "RTD5_RTD-" (at 224.79 105.41 180)
@@
     (pin "1")
   )
+  (symbol (lib_id "power:+3.3V") (at 274.32 48.26 0) (unit 1)
+    (in_bom yes) (on_board yes) (fields_autoplaced)
+    (property "Reference" "#PWR?" (id 0) (at 274.32 52.07 0)
+      (effects (font (size 1.27 1.27)) hide)
+    )
+    (property "Value" "+3.3V" (id 1) (at 274.32 43.18 0))
+    (property "Footprint" "" (id 2) (at 274.32 48.26 0)
+      (effects (font (size 1.27 1.27)) hide)
+    )
+    (property "Datasheet" "" (id 3) (at 274.32 48.26 0)
+      (effects (font (size 1.27 1.27)) hide)
+    )
+    (pin "1")
+  )
   (symbol (lib_id "MAX31865:MAX31865") (at 35.56 29.21 0) (unit 1)
     (in_bom yes) (on_board yes) (fields_autoplaced)
@@
     )
     (property "Datasheet" "~" (id 3) (at 261.62 156.972 0)
+      (effects (font (size 1.27 1.27)) hide)
+    )
+    (pin "1")
+  )
+  (symbol (lib_id "power:GND") (at 242.57 50.8 0) (unit 1)
+    (in_bom yes) (on_board yes) (fields_autoplaced)
+    (property "Reference" "#PWR?" (id 0) (at 242.57 57.15 0)
+      (effects (font (size 1.27 1.27)) hide)
+    )
+    (property "Value" "GND" (id 1) (at 242.57 55.88 0))
+    (property "Footprint" "" (id 2) (at 242.57 50.8 0)
+      (effects (font (size 1.27 1.27)) hide)
+    )
+    (property "Datasheet" "" (id 3) (at 242.57 50.8 0)
       (effects (font (size 1.27 1.27)) hide)
     )
@@
     (pin "1")
   )
+  (symbol (lib_id "power:GND") (at 270.51 50.8 0) (unit 1)
+    (in_bom yes) (on_board yes) (fields_autoplaced)
+    (property "Reference" "#PWR?" (id 0) (at 270.51 57.15 0)
+      (effects (font (size 1.27 1.27)) hide)
+    )
+    (property "Value" "GND" (id 1) (at 270.51 55.88 0))
+    (property "Footprint" "" (id 2) (at 270.51 50.8 0)
+      (effects (font (size 1.27 1.27)) hide)
+    )
+    (property "Datasheet" "" (id 3) (at 270.51 50.8 0)
+      (effects (font (size 1.27 1.27)) hide)
+    )
+    (pin "1")
+  )
   (symbol (lib_id "power:GND") (at 90.17 44.45 0) (unit 1)
     (in_bom yes) (on_board yes) (fields_autoplaced)
@@
     )
     (property "Datasheet" "" (id 3) (at 90.17 44.45 0)
+      (effects (font (size 1.27 1.27)) hide)
+    )
+    (pin "1")
+  )
+  (symbol (lib_id "power:+3.3V") (at 238.76 48.26 0) (unit 1)
+    (in_bom yes) (on_board yes) (fields_autoplaced)
+    (property "Reference" "#PWR?" (id 0) (at 238.76 52.07 0)
+      (effects (font (size 1.27 1.27)) hide)
+    )
+    (property "Value" "+3.3V" (id 1) (at 238.76 43.18 0))
+    (property "Footprint" "" (id 2) (at 238.76 48.26 0)
+      (effects (font (size 1.27 1.27)) hide)
+    )
+    (property "Datasheet" "" (id 3) (at 238.76 48.26 0)
       (effects (font (size 1.27 1.27)) hide)
     )
@@
     (pin "")
   )
+  (symbol (lib_id "power:GND") (at 251.46 59.69 0) (unit 1)
+    (in_bom yes) (on_board yes) (fields_autoplaced)
+    (property "Reference" "#PWR?" (id 0) (at 251.46 66.04 0)
+      (effects (font (size 1.27 1.27)) hide)
+    )
+    (property "Value" "GND" (id 1) (at 251.46 64.77 0))
+    (property "Footprint" "" (id 2) (at 251.46 59.69 0)
+      (effects (font (size 1.27 1.27)) hide)
+    )
+    (property "Datasheet" "" (id 3) (at 251.46 59.69 0)
+      (effects (font (size 1.27 1.27)) hide)
+    )
+    (pin "1")
+  )
   (symbol (lib_id "power:+3.3V") (at 175.26 85.09 0) (unit 1)
     (in_bom yes) (on_board yes) (fields_autoplaced)
@@
     )
     (property "Datasheet" "" (id 3) (at 193.04 58.42 0)
+      (effects (font (size 1.27 1.27)) hide)
+    )
+    (pin "1")
+  )
+  (symbol (lib_id "power:+3.3V") (at 275.59 62.23 0) (unit 1)
+    (in_bom yes) (on_board yes) (fields_autoplaced)
+    (property "Reference" "#PWR?" (id 0) (at 275.59 66.04 0)
+      (effects (font (size 1.27 1.27)) hide)
+    )
+    (property "Value" "+3.3V" (id 1) (at 275.59 57.15 0))
+    (property "Footprint" "" (id 2) (at 275.59 62.23 0)
+      (effects (font (size 1.27 1.27)) hide)
+    )
+    (property "Datasheet" "" (id 3) (at 275.59 62.23 0)
       (effects (font (size 1.27 1.27)) hide)
     )
@@
       (reference "#PWR?") (unit 1) (value "+3.3V") (footprint "")
     )
+    (path "/13ea1a53-08fd-4f09-b3eb-f1a7fa3c9c00"
+      (reference "#PWR?") (unit 1) (value "+3.3V") (footprint "")
+    )
+    (path "/16367de0-ecaf-47fd-aade-e34a3f2cc6b9"
+      (reference "#PWR?") (unit 1) (value "GND") (footprint "")
+    )
     (path "/18903017-2f04-4523-bdb1-ea26093fe55f"
       (reference "#PWR?") (unit 1) (value "GND") (footprint "")
@@
       (reference "#PWR?") (unit 1) (value "GND") (footprint "")
     )
+    (path "/3a983fc8-2c61-428f-9d9e-3a1f041e89e4"
+      (reference "#PWR?") (unit 1) (value "GND") (footprint "")
+    )
     (path "/4021a756-0e0d-427b-9bbb-f39cae2e98c8"
       (reference "#PWR?") (unit 1) (value "GND") (footprint "")
     )
+    (path "/47de8c2e-6067-4b89-88d4-59a79b5b8bb7"
+      (reference "#PWR?") (unit 1) (value "+3.3V") (footprint "")
+    )
     (path "/4dffbffc-699b-4e77-8084-f59d368983c2"
       (reference "#PWR?") (unit 1) (value "GND") (footprint "")
@@
       (reference "#PWR?") (unit 1) (value "GND") (footprint "")
     )
+    (path "/630cb47f-7b78-413f-8f9c-ee8578778e68"
+      (reference "#PWR?") (unit 1) (value "GND") (footprint "")
+    )
     (path "/669d4b70-b6d3-45a4-a586-dfab3e5d3dec"
       (reference "#PWR?") (unit 1) (value "+3.3V") (footprint "")
@@
       (reference "#PWR?") (unit 1) (value "GND") (footprint "")
     )
+    (path "/7bcd6448-6fe9-4ed4-afd9-d2514b6e0303"
+      (reference "#PWR?") (unit 1) (value "+3.3V") (footprint "")
+    )
     (path "/84393338-6440-4b3b-a0af-017f9f718a86"
