File: rtd_board/rtd_board.kicad_pcb (KiCad board)
At the start: 2 copper layers, 152.4 x 140 mm, 12 parts, among them J1 PCIE-LP-01-01-F-DV-A-TR, J7 DSUB1, J8 DSUB2, U1 MAX31865, U10 PCF8575_Breakout, U2 MAX31865, U3 MAX31865, U4 MAX31865, U5 MAX31865, U6 MAX31865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

Commit message: finishing up traces
Routing:
- net /IO_EXP_SC: track 0.00 -> 112.7 mm, vias 0 -> 1
- net /IO_EXP_SD: track 0.00 -> 109.3 mm, vias 0 -> 1
- net /SPI_SCK: track 254.7 -> 333.6 mm, vias 3 -> 4
- net /SPI_MOSI: track 290.0 -> 339.2 mm, vias 0 -> 1
- net /SPI_MISO: track 286.2 -> 334.7 mm
- net +3.3V: track 331.0 -> 371.7 mm
