File: core_board/core_board.kicad_sch (KiCad schematic)
At the start: 91 parts

Commit message: finished schematic
Parts:
- removed D?: D_Zener, symbol Device:D_Zener
- removed D?: D_Schottky, symbol Device:D_Schottky
- removed TP?: TestPoint, symbol Connector:TestPoint
- removed U?: MCP23017_Breakout, symbol MCP23017_Breakout:MCP23017_Breakout
- added C?: 100nF, symbol Device:C_Small
- added C?: 10uF, symbol Device:C_Small
- added D?: 40V, Diode_SMD:D_0603_1608Metric, symbol Device:D_Schottky
- added R? (x2): 10k, symbol Device:R_Small_US
- added R?: 1k, symbol Device:R_Small_US
- added TP?: TestPoint, symbol Connector:TestPoint
- added U?: PCF8575_Breakout, symbol PCF8575_Breakout:PCF8575_Breakout
- added U?: LD1117V33, TO255P1020X450X1968-3, symbol LD1117V33:LD1117V33
Connections:
- net +12V: now also J?.2 (Pin_2), D?.1 (K)
- net +3V3: now also U?.1 (VIN), C?.2, R?.1, R?.2, R?.2, U?.12 (VCC), U?.17 (VDD), U?.2 (VOUT), U?.9 (VDD); no longer C?.2, J?.A12, J?.A12, J?.A12, J?.A12, J?.A12, J?.A12, J?.A12, J?.A12, J?.A13, J?.A13, J?.A13, J?.A13, J?.A13, J?.A13, J?.A13, J?.A13, U?. (VIN), U?.2 (VOUT)
- net +5V: now also C?.2, U?.3 (VIN); no longer J?.B12, J?.B12, J?.B12, J?.B12, J?.B12, J?.B12, J?.B12, J?.B12, J?.B13, J?.B13, J?.B13, J?.B13, J?.B13, J?.B13, J?.B13, J?.B13
- net Button_0: now also U?.1 (P10)
- net Button_1: now also U?.2 (P11)
- net Button_2: now also U?.3 (P12)
- net Button_3: now also U?.4 (P13)
- net Button_4: now also U?.5 (P14)
- net Button_5: now also U?.6 (P15)
- net Button_6: now also U?.7 (P16)
- net Button_7: now also U?.8 (P17)
- net GND: now also U?.2 (GND), U?.6 (A0), U?.7 (A1), U?.8 (A2), C?.1, C?.1, D?.2 (A), U?.1 (ADJ/GND), U?.10 (GND), U?.11 (GND), U?.16 (GND); no longer U?. (VIN)
- net I2C_SCL_0: now also U?.10 (SC0); no longer U?. (VIN)
- net I2C_SCL_1: now also U?.12 (SC1); no longer U?. (VIN)
- net I2C_SCL_2: now also U?.14 (SC2); no longer U?. (VIN)
- net I2C_SCL_3: now also U?.16 (SC3); no longer U?. (VIN)
- net I2C_SCL_4: now also U?.18 (SC4); no longer U?. (VIN)
- net I2C_SCL_5: now also U?.20 (SC5); no longer U?. (VIN)
- net I2C_SCL_6: now also U?.22 (SC6); no longer U?. (VIN)
- net I2C_SCL_7: now also U?.24 (SC7); no longer U?. (VIN)
- net I2C_SCL_SLOW: now also U?.4 (SCL), U?.14 (SCL); no longer U?. (VIN)
- net I2C_SDA_0: now also U?.9 (SD0); no longer U?. (VIN)
- net I2C_SDA_1: now also U?.11 (SD1); no longer U?. (VIN)
- net I2C_SDA_2: now also U?.13 (SD2); no longer U?. (VIN)
- net I2C_SDA_3: now also U?.15 (SD3); no longer U?. (VIN)
- net I2C_SDA_4: now also U?.17 (SD4); no longer U?. (VIN)
- net I2C_SDA_5: now also U?.19 (SD5); no longer U?. (VIN)
- net I2C_SDA_6: now also U?.21 (SD6); no longer U?. (VIN)
- net I2C_SDA_7: now also U?.23 (SD7); no longer U?. (VIN)
- net I2C_SDA_SLOW: now also U?.3 (SDA), U?.13 (SDA); no longer U?. (VIN)
- net INT: now also R?.2, U?.15 (INT)
- net LED_0: now also U?.18 (P00)
- net LED_1: now also U?.19 (P01)
- net LED_2: now also U?.20 (P02)
- net LED_3: now also U?.21 (P03)
- net LED_4: now also U?.22 (P04)
- net LED_5: now also U?.23 (P05)
- net LED_6: now also U?.24 (P06)
- net LED_7: now also U?.25 (P07)
- net at TP?.1, U?.1 (CD): now also R?.1
- net at U?.1 (CD): now also R?.1, TP?.1
- net buck_converter1/V_OUT renamed EXT_5V
- net EXT_5V: now also J?.B12, J?.B12, J?.B12, J?.B12, J?.B12, J?.B12, J?.B12, J?.B12, J?.B13, J?.B13, J?.B13, J?.B13, J?.B13, J?.B13, J?.B13, J?.B13
- new net EXT_3V3: C?.2, J?.A12, J?.A12, J?.A12, J?.A12, J?.A12, J?.A12, J?.A12, J?.A12, J?.A13, J?.A13, J?.A13, J?.A13, J?.A13, J?.A13, J?.A13, J?.A13, U?.2 (VOUT)
- no-connect marks 10 -> 8
Other:
- removed sheet buck_converter
- added sheet buck_converter2 (buck_converter.kicad_sch)
- moved on the sheet: C?, D?, J?, JP?, R?, SW?, TP?, U?
