File: core_board/core_board.kicad_pcb (KiCad board)
At the start: 2 copper layers, 355.6 x 152.4 mm, 127 parts, among them J1 Conn_01x02, J10 PCIE-LP-01-01-F-DV-A-TR, J2 UART Pins, J3 PCIE-LP-01-01-F-DV-A-TR, J4 PCIE-LP-01-01-F-DV-A-TR, J5 PCIE-LP-01-01-F-DV-A-TR, J6 PCIE-LP-01-01-F-DV-A-TR, J7 PCIE-LP-01-01-F-DV-A-TR, J8 PCIE-LP-01-01-F-DV-A-TR, J9 PCIE-LP-01-01-F-DV-A-TR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

Commit message: more routing progress
Parts:
- removed TP1, TP2: TestPoint, TestPoint:TestPoint_Plated_Hole_D2.0mm
- moved R1 58.6 mm to (164.3, 252.2), turned to 90 degrees
- moved R2 55.2 mm to (161.3, 252.2), turned to 90 degrees
- moved R31 48.4 mm to (254.5, 204.0)
- moved R5 48.4 mm to (254.5, 215.6)
- moved R15 48.4 mm to (262.4, 222.0)
- moved R20 48.4 mm to (254.5, 207.5)
- moved R24 48.4 mm to (254.5, 210.1)
- moved R27 48.4 mm to (262.4, 207.5)
- moved R30 48.4 mm to (254.5, 221.2)
- moved R34 48.4 mm to (254.5, 212.6)
- moved R35 48.4 mm to (254.5, 224.3)
- moved R4 48.4 mm to (262.6, 215.9)
- moved R8 48.4 mm to (250.7, 227.6)
- moved R16 48.4 mm to (250.5, 204.0)
- moved R10 48.4 mm to (250.4, 221.0)
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Routing:
- net /SPI_CS_CORE: track 0.00 -> 249.1 mm, vias 0 -> 2
- net /SPI_SCK_CORE: track 0.00 -> 240.8 mm, vias 0 -> 4
- net /SPI_MISO_CORE: track 0.00 -> 231.5 mm, vias 0 -> 4
- net /I2C_SDA_SLOW: track 0.00 -> 211.3 mm, vias 0 -> 1
- net /SPI_MOSI_CORE: track 0.00 -> 197.2 mm, vias 0 -> 4
- net /I2C_SCL_SLOW: track 0.00 -> 181.6 mm, vias 0 -> 1
- net /SPI_CS_1: track 0.00 -> 151.9 mm
- net /SPI_CS_2: track 0.00 -> 150.2 mm
- net /SPI_SCK: track 0.00 -> 148.5 mm
- net /SPI_MOSI: track 0.00 -> 147.7 mm
- net /SPI_MISO: track 0.00 -> 147.6 mm
- net /SPI_CS_0: track 0.00 -> 134.7 mm
- net /I2C_SDA_FAST: track 0.00 -> 105.2 mm
- net /I2C_SCL_FAST: track 0.00 -> 98.1 mm
- net Net-(JP3-Pad3): track 0.00 -> 58.3 mm, vias 0 -> 2
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Other:
- board text added: "RX"
- board text added: "TX"

Commit message: more routing
Parts:
- moved R4 145.2 mm to (133.3, 149.9), turned to -90 degrees
- moved R5 131.2 mm to (141.0, 149.9), turned to -90 degrees
- moved R6 130.4 mm to (148.6, 149.9), turned to -90 degrees
- moved R8 116.6 mm to (163.8, 149.9), turned to -90 degrees
- moved R7 110.5 mm to (156.2, 149.9), turned to -90 degrees
- moved R10 106.3 mm to (171.4, 149.9), turned to -90 degrees
- moved R14 105.6 mm to (186.7, 149.9), turned to -90 degrees
- moved R11 101.9 mm to (179.1, 149.9), turned to -90 degrees
- moved R9 7.60 mm to (246.6, 206.0)
Routing:
- net /EXT_3V3: track 599.1 -> 450.6 mm
- net /INT: track 0.00 -> 131.0 mm, vias 0 -> 2
- net /Button_0: track 0.00 -> 103.0 mm, vias 0 -> 2
- net /Button_2: track 0.00 -> 92.4 mm
- net /Button_1: track 0.00 -> 92.2 mm, vias 0 -> 2
- net /Button_3: track 0.00 -> 81.0 mm
- net /Button_4: track 0.00 -> 69.6 mm
- net /LED_0: track 0.00 -> 66.0 mm, vias 0 -> 1
- net /LED_4: track 0.00 -> 61.2 mm, vias 0 -> 1
- net /Button_5: track 0.00 -> 58.0 mm
- net /LED_1: track 0.00 -> 57.0 mm, vias 0 -> 1
- net /LED_5: track 0.00 -> 55.6 mm, vias 0 -> 1
- net /LED_6: track 0.00 -> 49.9 mm, vias 0 -> 1
- net /LED_2: track 0.00 -> 48.0 mm, vias 0 -> 1
- net /LED_7: track 0.00 -> 45.3 mm, vias 0 -> 1
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
Commit message: more routing
Parts:
- moved J6 0.10 mm to (331.2, 274.3)
- moved J7 0.10 mm to (366.8, 274.3)
- moved J8 0.10 mm to (402.3, 274.3)
Routing:
- net /BROADCAST: track 0.00 -> 717.9 mm, vias 0 -> 10
- net /SPI_MOSI: track 147.7 -> 730.4 mm, vias 0 -> 25
- net /SPI_SCK: track 148.5 -> 722.6 mm, vias 0 -> 25
- net /SPI_MISO: track 147.6 -> 717.9 mm, vias 0 -> 25
- net /SPI_CS_2: track 150.2 -> 704.1 mm, vias 0 -> 25
- net /SPI_CS_1: track 151.9 -> 700.4 mm, vias 0 -> 25
- net /SPI_CS_0: track 134.7 -> 674.1 mm, vias 0 -> 9
- net /I2C_SCL_FAST: track 98.1 -> 602.2 mm, vias 0 -> 9
- net /I2C_SDA_FAST: track 105.2 -> 601.5 mm, vias 0 -> 9
- net /EXT_5V: track 502.2 -> 42.9 mm, vias 0 -> 8
- net +5V: track 156.3 -> 24.8 mm
- net /EXT_3V3: track 450.6 -> 441.2 mm
- net +3V3: track 246.6 -> 251.0 mm
- net Net-(JP1-Pad2): track 82.0 -> 80.1 mm
- net Net-(JP3-Pad3): vias 2 -> 0
