File: core_board/buck_converter.kicad_sch (KiCad schematic)
At the start: 16 parts

Commit message: created netlist
Parts:
- C12, C13, C16, C17, C18: renamed from C?; footprint (none) -> Capacitor_SMD:C_0603_1608Metric
- C14, C15: renamed from C?; footprint (none) -> Capacitor_SMD:C_1206_3216Metric
- L2: renamed from L?; footprint (none) -> Inductor_SMD:L_Bourns_SRP5030T
- R45, R46, R47, R48, R49, R50: renamed from R?; footprint (none) -> Resistor_SMD:R_0603_1608Metric
- U9: renamed from U?; footprint VREG_LM5017MR/NOPB -> TPS54332DDAR:VREG_LM5017MR_NOPB
- gave numbers to parts that had none: 1
Changed lines of the file:
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@@
   (symbol (lib_id "Device:R_Small_US") (at 140.462 78.994 270)
     (in_bom yes) (on_board yes)
-    (property "Reference" "R?" (id 0) (at 140.462 83.566 90))
+    (property "Reference" "R48" (id 0) (at 140.462 83.566 90))
     (property "Value" "10k" (id 1) (at 140.462 81.534 90))
-    (property "Footprint" "" (id 2) (at 140.462 78.994 0)
+    (property "Footprint" "Resistor_SMD:R_0603_1608Metric" (id 2) (at 140.462 78.994 0)
       (effects (font (size 1.27 1.27)) hide)
     )
@@
   (symbol (lib_id "Device:L_Small") (at 131.318 85.09 180)
     (in_bom yes) (on_board yes) (fields_autoplaced)
-    (property "Reference" "L?" (id 0) (at 132.842 83.8199 0)
+    (property "Reference" "L2" (id 0) (at 132.842 83.8199 0)
       (effects (font (size 1.27 1.27)) (justify right))
     )
@@
       (effects (font (size 1.27 1.27)) (justify right))
     )
-    (property "Footprint" "" (id 2) (at 131.318 85.09 0)
+    (property "Footprint" "Inductor_SMD:L_Bourns_SRP5030T" (id 2) (at 131.318 85.09 0)
       (effects (font (size 1.27 1.27)) hide)
     )
@@
   (symbol (lib_id "Device:C_Small") (at 140.462 64.008 90)
     (in_bom yes) (on_board yes)
-    (property "Reference" "C?" (id 0) (at 139.192 67.056 90)
+    (property "Reference" "C14" (id 0) (at 139.192 67.056 90)
       (effects (font (size 1.27 1.27)) (justify left))
     )
@@
       (effects (font (size 1.27 1.27)) (justify left))
     )
-    (property "Footprint" "" (id 2) (at 140.462 64.008 0)
+    (property "Footprint" "Capacitor_SMD:C_1206_3216Metric" (id 2) (at 140.462 64.008 0)
       (effects (font (size 1.27 1.27)) hide)
     )
@@
   (symbol (lib_id "Device:C_Small") (at 140.716 102.362 0)
     (in_bom yes) (on_board yes)
-    (property "Reference" "C?" (id 0) (at 132.08 101.092 0)
+    (property "Reference" "C16" (id 0) (at 132.08 101.092 0)
       (effects (font (size 1.27 1.27)) (justify left))
     )
@@
       (effects (font (size 1.27 1.27)) (justify left))
     )
-    (property "Footprint" "" (id 2) (at 140.716 102.362 0)
+    (property "Footprint" "Capacitor_SMD:C_0603_1608Metric" (id 2) (at 140.716 102.362 0)
       (effects (font (size 1.27 1.27)) hide)
     )
@@
   (symbol (lib_id "Device:R_Small_US") (at 150.876 78.994 270)
     (in_bom yes) (on_board yes)
-    (property "Reference" "R?" (id 0) (at 150.876 83.566 90))
+    (property "Reference" "R49" (id 0) (at 150.876 83.566 90))
     (property "Value" "1.9k" (id 1) (at 150.876 81.534 90))
-    (property "Footprint" "" (id 2) (at 150.876 78.994 0)
+    (property "Footprint" "Resistor_SMD:R_0603_1608Metric" (id 2) (at 150.876 78.994 0)
       (effects (font (size 1.27 1.27)) hide)
     )
@@
   (symbol (lib_id "Device:C_Small") (at 185.674 98.044 180)
     (in_bom yes) (on_board yes)
-    (property "Reference" "C?" (id 0) (at 188.722 99.314 90)
+    (property "Reference" "C17" (id 0) (at 188.722 99.314 90)
       (effects (font (size 1.27 1.27)) (justify left))
     )
@@
       (effects (font (size 1.27 1.27)) (justify left))
     )
-    (property "Footprint" "" (id 2) (at 185.674 98.044 0)
+    (property "Footprint" "Capacitor_SMD:C_0603_1608Metric" (id 2) (at 185.674 98.044 0)
       (effects (font (size 1.27 1.27)) hide)
     )
@@
   (symbol (lib_id "Device:R_Small_US") (at 95.504 91.186 180)
     (in_bom yes) (on_board yes)
-    (property "Reference" "R?" (id 0) (at 90.932 91.186 90))
+    (property "Reference" "R46" (id 0) (at 90.932 91.186 90))
     (property "Value" "50k" (id 1) (at 92.964 91.186 90))
-    (property "Footprint" "" (id 2) (at 95.504 91.186 0)
+    (property "Footprint" "Resistor_SMD:R_0603_1608Metric" (id 2) (at 95.504 91.186 0)
       (effects (font (size 1.27 1.27)) hide)
     )
@@
   (symbol (lib_id "power:GND") (at 197.358 116.586 0)
     (in_bom yes) (on_board yes) (fields_autoplaced)
-    (property "Reference" "#PWR?" (id 0) (at 197.358 122.936 0)
+    (property "Reference" "#PWR097" (id 0) (at 197.358 122.936 0)
       (effects (font (size 1.27 1.27)) hide)
     )
@@
   (symbol (lib_id "Device:R_Small_US") (at 107.188 90.424 90)
     (in_bom yes) (on_board yes)
-    (property "Reference" "R?" (id 0) (at 104.902 92.71 90))
+    (property "Reference" "R47" (id 0) (at 104.902 92.71 90))
     (property "Value" "1M" (id 1) (at 108.712 92.71 90))
-    (property "Footprint" "" (id 2) (at 107.188 90.424 0)
+    (property "Footprint" "Resistor_SMD:R_0603_1608Metric" (id 2) (at 107.188 90.424 0)
       (effects (font (size 1.27 1.27)) hide)
     )
@@
   (symbol (lib_id "power:GND") (at 159.766 78.994 0)
     (in_bom yes) (on_board yes) (fields_autoplaced)
-    (property "Reference" "#PWR?" (id 0) (at 159.766 85.344 0)
+    (property "Reference" "#PWR096" (id 0) (at 159.766 85.344 0)
       (effects (font (size 1.27 1.27)) hide)
     )
@@
   (symbol (lib_id "Device:C_Small") (at 107.188 96.266 90)
     (in_bom yes) (on_board yes)
-    (property "Reference" "C?" (id 0) (at 105.918 99.314 90)
+    (property "Reference" "C13" (id 0) (at 105.918 99.314 90)
       (effects (font (size 1.27 1.27)) (justify left))
     )
@@
       (effects (font (size 1.27 1.27)) (justify left))
     )
-    (property "Footprint" "" (id 2) (at 107.188 96.266 0)
+    (property "Footprint" "Capacitor_SMD:C_0603_1608Metric" (id 2) (at 107.188 96.266 0)
       (effects (font (size 1.27 1.27)) hide)
     )
@@
   (symbol (lib_id "Device:R_Small_US") (at 193.548 108.458 0)
     (in_bom yes) (on_board yes)
-    (property "Reference" "R?" (id 0) (at 198.12 108.458 90))
+    (property "Reference" "R50" (id 0) (at 198.12 108.458 90))
     (property "Value" "150k" (id 1) (at 196.088 108.458 90))
-    (property "Footprint" "" (id 2) (at 193.548 108.458 0)
+    (property "Footprint" "Resistor_SMD:R_0603_1608Metric" (id 2) (at 193.548 108.458 0)
       (effects (font (size 1.27 1.27)) hide)
     )
@@
   (symbol (lib_id "power:GND") (at 81.788 96.266 0)
     (in_bom yes) (on_board yes) (fields_autoplaced)
-    (property "Reference" "#PWR?" (id 0) (at 81.788 102.616 0)
+    (property "Reference" "#PWR094" (id 0) (at 81.788 102.616 0)
       (effects (font (size 1.27 1.27)) hide)
     )
@@
   (symbol (lib_id "power:GND") (at 118.11 111.506 0)
     (in_bom yes) (on_board yes) (fields_autoplaced)
-    (property "Reference" "#PWR?" (id 0) (at 118.11 117.856 0)
+    (property "Reference" "#PWR095" (id 0) (at 118.11 117.856 0)
       (effects (font (size 1.27 1.27)) hide)
     )
@@
   (symbol (lib_id "Device:C_Small") (at 86.106 87.376 0)
     (in_bom yes) (on_board yes)
-    (property "Reference" "C?" (id 0) (at 77.47 86.106 0)
+    (property "Reference" "C12" (id 0) (at 77.47 86.106 0)
       (effects (font (size 1.27 1.27)) (justify left))
     )
@@
       (effects (font (size 1.27 1.27)) (justify left))
     )
-    (property "Footprint" "" (id 2) (at 86.106 87.376 0)
+    (property "Footprint" "Capacitor_SMD:C_0603_1608Metric" (id 2) (at 86.106 87.376 0)
       (effects (font (size 1.27 1.27)) hide)
     )
@@
   (symbol (lib_id "Diode:B340") (at 122.428 105.156 270)
     (in_bom yes) (on_board yes) (fields_autoplaced)
-    (property "Reference" "D?" (id 0) (at 125.222 103.5684 90)
+    (property "Reference" "D11" (id 0) (at 125.222 103.5684 90)
       (effects (font (size 1.27 1.27)) (justify left))
     )
@@
   (symbol (lib_id "Device:C_Small") (at 193.548 98.044 180)
     (in_bom yes) (on_board yes)
-    (property "Reference" "C?" (id 0) (at 196.596 99.314 90)
+    (property "Reference" "C18" (id 0) (at 196.596 99.314 90)
       (effects (font (size 1.27 1.27)) (justify left))
     )
@@
       (effects (font (size 1.27 1.27)) (justify left))
     )
-    (property "Footprint" "" (id 2) (at 193.548 98.044 0)
+    (property "Footprint" "Capacitor_SMD:C_0603_1608Metric" (id 2) (at 193.548 98.044 0)
       (effects (font (size 1.27 1.27)) hide)
     )
@@
   (symbol (lib_id "Device:R_Small_US") (at 95.504 83.566 180)
     (in_bom yes) (on_board yes)
-    (property "Reference" "R?" (id 0) (at 90.932 83.566 90))
+    (property "Reference" "R45" (id 0) (at 90.932 83.566 90))
     (property "Value" "150k" (id 1) (at 92.964 83.566 90))
-    (property "Footprint" "" (id 2) (at 95.504 83.566 0)
+    (property "Footprint" "Resistor_SMD:R_0603_1608Metric" (id 2) (at 95.504 83.566 0)
       (effects (font (size 1.27 1.27)) hide)
     )
@@
   (symbol (lib_id "TPS54332DDAR:TPS54332DDAR") (at 164.846 103.886 0)
     (in_bom yes) (on_board yes)
-    (property "Reference" "U?" (id 0) (at 153.162 86.614 0))
+    (property "Reference" "U9" (id 0) (at 153.162 86.614 0))
     (property "Value" "TPS54332DDAR" (id 1) (at 170.434 86.614 0))
-    (property "Footprint" "VREG_LM5017MR/NOPB" (id 2) (at 164.846 103.886 0)
+    (property "Footprint" "TPS54332DDAR:VREG_LM5017MR_NOPB" (id 2) (at 164.846 103.886 0)
       (effects (font (size 1.27 1.27)) (justify left bottom) hide)
     )
@@
   (symbol (lib_id "Device:C_Small") (at 140.462 71.628 90)
     (in_bom yes) (on_board yes)
-    (property "Reference" "C?" (id 0) (at 139.192 74.676 90)
+    (property "Reference" "C15" (id 0) (at 139.192 74.676 90)
       (effects (font (size 1.27 1.27)) (justify left))
     )
@@
       (effects (font (size 1.27 1.27)) (justify left))
     )
-    (property "Footprint" "" (id 2) (at 140.462 71.628 0)
-      (effects (font (size 1.27 1.27)) hide)
-    )
+    (property "Footprint" "Capacitor_SMD:C_1206_3216Metric" (id 2) (at 140.462 71.628 0)
+      (effects (font (size 1.27 1.27)) hide)
+    )

Commit message: small edits to power supply
Parts:
- D11: footprint Diode_SMD:D_SMC -> Diode_SMD:D_SMA
Changed lines of the file:
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@@
       (effects (font (size 1.27 1.27)) (justify left))
     )
-    (property "Footprint" "Diode_SMD:D_SMC" (id 2) (at 117.983 105.156 0)
+    (property "Footprint" "Diode_SMD:D_SMA" (id 2) (at 117.983 105.156 0)
       (effects (font (size 1.27 1.27)) hide)
     )
